File: pcb/KB426/KB426.kicad_pcb (KiCad board)
At the start: 2 copper layers, 129 parts, among them SW1 SW_Push_45deg, SW10 SW_Push_45deg, SW11 SW_Push_45deg, SW12 SW_Push_45deg, SW13 SW_Push_45deg, SW14 SW_Push_45deg, SW15 SW_Push_45deg, SW16 SW_Push_45deg, SW17 SW_Push_45deg, SW18 SW_Push_45deg, SW19 SW_Push_45deg, SW2 SW_Push_45deg, SW20 SW_Push_45deg, SW21 SW_Push_45deg, SW22 SW_Push_45deg, SW23 SW_Push_45deg, SW24 SW_Push_45deg, SW25 SW_Push_45deg, SW26 SW_Push_45deg, SW27 SW_Push_45deg, SW28 SW_Push_45deg, SW29 SW_Push_45deg, SW3 SW_Push_45deg, SW30 SW_Push_45deg, SW31 SW_Push_45deg, SW32 SW_Push_45deg, SW33 SW_Push_45deg, SW34 SW_Push_45deg, SW35 SW_Push_45deg, SW36 SW_Push_45deg, SW37 SW_Push_45deg, SW38 SW_Push_45deg, SW39 SW_Push_45deg, SW4 SW_Push_45deg, SW40 SW_Push_45deg, SW41 SW_Push_45deg, SW42 SW_Push_45deg, SW43 SW_Push_45deg, SW44 SW_Push_45deg, SW45 SW_Push_45deg, SW46 SW_Push_45deg, SW47 SW_Push_45deg, SW48 SW_Push_45deg, SW49 SW_Push_45deg, SW5 SW_Push_45deg, SW50 SW_Push_45deg, SW51 SW_Push_45deg, SW52 SW_Push_45deg, SW53 SW_Push_45deg, SW54 SW_Push_45deg, SW55 SW_Push_45deg, SW56 SW_Push_45deg, SW57 SW_Push_45deg, SW58 SW_Push_45deg, SW59 SW_Push_45deg, SW6 SW_Push_45deg, SW60 SW_Push_45deg, SW61 SW_Push_45deg, SW62 SW_Push_45deg, SW63 SW_Push_45deg, SW64 SW_Push_45deg, SW7 SW_Push_45deg, SW8 SW_Push_45deg, SW9 SW_Push_45deg, U1 Pico

Commit message: + update pcb
Parts:
- moved D53 162.6 mm to (314.3, 138.7)
- moved D9 159.3 mm to (85.7, 138.7)
- moved D54 150.1 mm to (333.4, 138.7)
- moved D10 144.6 mm to (104.8, 138.7)
- moved D11 130.0 mm to (123.8, 138.7)
- moved D46 118.8 mm to (333.4, 119.6)
- moved D26 117.3 mm to (367.7, 60.3)
- moved D39 117.3 mm to (367.7, 49.5)
- moved D12 115.7 mm to (142.9, 138.7)
- moved D2 111.9 mm to (104.8, 119.6)
- moved D45 105.7 mm to (314.3, 119.6)
- moved D25 103.0 mm to (349.6, 60.4)
- moved D38 103.0 mm to (349.6, 49.7)
- moved D64 103.0 mm to (349.6, 28.1)
- moved D13 101.7 mm to (161.9, 138.7)
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Routing:
- net Net-(D52-A): track 0.00 -> 5.84 mm
- net Net-(D53-A): track 0.00 -> 5.81 mm
- net Net-(D45-A): track 0.00 -> 5.81 mm
- net Net-(D44-A): track 0.00 -> 5.81 mm
- net Net-(D16-A): track 0.00 -> 5.81 mm
- net Net-(D9-A): track 0.00 -> 5.81 mm
- net Net-(D49-A): track 0.00 -> 5.81 mm
- net Net-(D15-A): track 0.00 -> 5.81 mm
- net Net-(D14-A): track 0.00 -> 5.81 mm
- net Net-(D12-A): track 0.00 -> 5.81 mm
- net Net-(D8-A): track 0.00 -> 5.81 mm
- net Net-(D11-A): track 0.00 -> 5.81 mm
- net Net-(D1-A): track 0.00 -> 5.81 mm
- net Net-(D7-A): track 0.00 -> 5.81 mm
- net Net-(D6-A): track 0.00 -> 5.81 mm
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
Commit message: + update pcb
Parts:
- moved D25 288.4 mm to (85.7, 176.8)
- moved D26 287.6 mm to (104.8, 176.8)
- moved D33 231.2 mm to (85.7, 195.8)
- moved D34 228.1 mm to (104.8, 195.8)
- moved D35 221.7 mm to (123.8, 195.8)
- moved D36 219.5 mm to (142.9, 195.8)
- moved D40 204.7 mm to (314.7, 195.0)
- moved D55 182.1 mm to (314.2, 176.4)
- moved D64 174.0 mm to (257.0, 175.5)
- moved D17 171.3 mm to (85.7, 157.7)
- moved D18 166.4 mm to (104.8, 157.7)
- moved D37 166.4 mm to (257.2, 195.1)
- moved D38 163.4 mm to (276.0, 195.5)
- moved D39 162.6 mm to (295.4, 195.2)
- moved D48 160.7 mm to (333.1, 195.1)
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Routing:
- net Net-(D61-A): track 0.00 -> 5.81 mm
- net Net-(D60-A): track 0.00 -> 5.81 mm
- net Net-(D24-A): track 0.00 -> 5.81 mm
- net Net-(D17-A): track 0.00 -> 5.81 mm
- net Net-(D57-A): track 0.00 -> 5.81 mm
- net Net-(D23-A): track 0.00 -> 5.81 mm
- net Net-(D22-A): track 0.00 -> 5.81 mm
- net Net-(D20-A): track 0.00 -> 5.81 mm
- net Net-(D19-A): track 0.00 -> 5.81 mm
- net Net-(D18-A): track 0.00 -> 5.81 mm
- net Net-(D62-A): track 0.00 -> 5.81 mm
- net Net-(D21-A): track 0.00 -> 5.81 mm
- net Net-(D59-A): track 0.00 -> 5.81 mm
- net Net-(D58-A): track 0.00 -> 5.81 mm

Commit message: + update pcb
Parts:
- moved D36 47.5 mm to (190.4, 195.8)
- moved D47 9.75 mm to (285.9, 176.7)
- moved U1 3.79 mm to (111.9, 72.7)
- moved D64 1.32 mm to (257.2, 176.8)
- moved D63 1.24 mm to (333.4, 176.8)
- moved D40 0.94 mm to (314.3, 195.8)
- moved D48 0.80 mm to (333.4, 195.8)
- moved D37 0.70 mm to (257.2, 195.8)
- moved D32 0.65 mm to (219.1, 176.8)
- moved D39 0.63 mm to (295.3, 195.8)
- moved D30 0.49 mm to (181.0, 176.8)
- moved D56 0.46 mm to (238.1, 176.8)
- moved D31 0.44 mm to (200.0, 176.8)
- moved D38 0.40 mm to (276.2, 195.8)
- moved D55 0.35 mm to (314.3, 176.8)
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Routing:
- net Column 3: track 0.00 -> 323.2 mm
- net Row 4: track 0.00 -> 228.6 mm
- net Column 5: track 0.00 -> 205.9 mm
- net Column 4: track 0.00 -> 205.3 mm
- net Row 5: track 0.00 -> 168.7 mm
- net Row 6: track 0.00 -> 159.9 mm
- net Row 3: track 0.00 -> 133.3 mm
- net Row 2: track 0.00 -> 133.3 mm
- net Row 1: track 0.00 -> 133.3 mm
- net Row 0: track 0.00 -> 133.3 mm
- net Row 7: track 0.00 -> 116.4 mm
- net Column 2: track 0.00 -> 114.3 mm
- net Column 1: track 0.00 -> 114.3 mm
- net Column 0: track 0.00 -> 114.3 mm
- net Column 7: track 0.00 -> 57.2 mm
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
Commit message: + update sch and pcb
Parts:
- SW47: footprint PCM_Switch_Keyboard_Cherry_MX:SW_Cherry_MX_PCB_2.00u -> PCM_Switch_Keyboard_Cherry_MX:SW_Cherry_MX_PCB_1.00u
- SW56: footprint PCM_Switch_Keyboard_Cherry_MX:SW_Cherry_MX_PCB_1.00u -> PCM_Switch_Keyboard_Cherry_MX:SW_Cherry_MX_PCB_2.00u
- moved D63 95.2 mm to (238.1, 176.8)
- moved SW63 95.2 mm to (247.7, 171.4)
- moved D56 66.7 mm to (304.8, 176.8)
- moved SW56 66.7 mm to (314.3, 171.4)
- moved SW47 47.6 mm to (342.9, 171.4)
- moved D47 47.5 mm to (333.4, 176.8)
- moved SW55 38.1 mm to (285.8, 171.4)
- moved D55 38.1 mm to (276.2, 176.8)
- moved U1 13.4 mm to (111.4, 86.1)
Connections:
- net Column 0 renamed Net-(U1-GPIO8)
- net Column 1 renamed Net-(U1-GPIO9)
- net Column 2 renamed Net-(U1-GPIO10)
- net Column 3 renamed Net-(U1-GPIO11)
- net Column 4 renamed Net-(U1-GPIO12)
- net Column 5 renamed Net-(U1-GPIO13)
- net Row 2 renamed Net-(D17-K)
- net Row 6 renamed Net-(D49-K)
- D1 pad 1: Row 0 -> Net-(D1-K)
- D10 pad 1: Row 1 -> Net-(D10-K)
- D11 pad 1: Row 1 -> Net-(D10-K)
- D12 pad 1: Row 1 -> Net-(D10-K)
- D13 pad 1: Row 1 -> Net-(D10-K)
- D14 pad 1: Row 1 -> Net-(D10-K)
- D15 pad 1: Row 1 -> Net-(D10-K)
- D16 pad 1: Row 1 -> Net-(D10-K)
- D2 pad 1: Row 0 -> Net-(D1-K)
- D25 pad 1: Row 3 -> Net-(D25-K)
- D26 pad 1: Row 3 -> Net-(D25-K)
- D27 pad 1: Row 3 -> Net-(D25-K)
- D28 pad 1: Row 3 -> Net-(D25-K)
- D29 pad 1: Row 3 -> Net-(D25-K)
- D3 pad 1: Row 0 -> Net-(D1-K)
- D30 pad 1: Row 3 -> Net-(D25-K)
- D31 pad 1: Row 3 -> Net-(D25-K)
- D32 pad 1: Row 3 -> Net-(D25-K)
- D33 pad 1: Row 4 -> Net-(D33-K)
- D34 pad 1: Row 4 -> Net-(D33-K)
- D35 pad 1: Row 4 -> Net-(D33-K)
- D36 pad 1: Row 4 -> Net-(D33-K)
- D37 pad 1: Row 4 -> Net-(D33-K)
- D38 pad 1: Row 4 -> Net-(D33-K)
- D39 pad 1: Row 4 -> Net-(D33-K)
- D4 pad 1: Row 0 -> Net-(D1-K)
- D40 pad 1: Row 4 -> Net-(D33-K)
- D41 pad 1: Row 5 -> Net-(D41-K)
- D42 pad 1: Row 5 -> Net-(D41-K)
- D43 pad 1: Row 5 -> Net-(D41-K)
- D44 pad 1: Row 5 -> Net-(D41-K)
- D45 pad 1: Row 5 -> Net-(D41-K)
- D46 pad 1: Row 5 -> Net-(D41-K)
- D47 pad 1: Row 5 -> Net-(D41-K)
- D48 pad 1: Row 5 -> Net-(D41-K)
- D5 pad 1: Row 0 -> Net-(D1-K)
- D57 pad 1: Row 7 -> Net-(D57-K)
- D58 pad 1: Row 7 -> Net-(D57-K)
- D59 pad 1: Row 7 -> Net-(D57-K)
- D6 pad 1: Row 0 -> Net-(D1-K)
- D60 pad 1: Row 7 -> Net-(D57-K)
- D61 pad 1: Row 7 -> Net-(D57-K)
- D62 pad 1: Row 7 -> Net-(D57-K)
- D63 pad 1: Row 7 -> Net-(D57-K)
- D64 pad 1: Row 7 -> Net-(D57-K)
- D7 pad 1: Row 0 -> Net-(D1-K)
- D8 pad 1: Row 0 -> Net-(D1-K)
- D9 pad 1: Row 1 -> Net-(D10-K)
- SW15 pad 2: Column 6 -> Net-(U1-GPIO14)
- SW16 pad 2: Column 7 -> Net-(U1-GPIO15)
- SW23 pad 2: Column 6 -> Net-(U1-GPIO14)
- SW24 pad 2: Column 7 -> Net-(U1-GPIO15)
- SW31 pad 2: Column 6 -> Net-(U1-GPIO14)
- SW32 pad 2: Column 7 -> Net-(U1-GPIO15)
- SW39 pad 2: Column 6 -> Net-(U1-GPIO14)
- SW40 pad 2: Column 7 -> Net-(U1-GPIO15)
- SW47 pad 2: Column 7 -> Net-(U1-GPIO14)
- SW48 pad 2: Column 6 -> Net-(U1-GPIO15)
- SW55 pad 2: Column 7 -> Net-(U1-GPIO14)
- SW56 pad 2: Column 6 -> Net-(U1-GPIO15)
- SW63 pad 2: Column 7 -> Net-(U1-GPIO14)
- SW64 pad 2: Column 6 -> Net-(U1-GPIO15)
- SW7 pad 2: Column 6 -> Net-(U1-GPIO14)
- SW8 pad 2: Column 7 -> Net-(U1-GPIO15)
- U1 pad 1: Row 0 -> Net-(D33-K)
- U1 pad 10: Row 7 -> Net-(D41-K)
- U1 pad 19: Column 6 -> Net-(U1-GPIO14)
- U1 pad 2: Row 1 -> Net-(D25-K)
- U1 pad 20: Column 7 -> Net-(U1-GPIO15)
- U1 pad 5: Row 3 -> Net-(D10-K)
- U1 pad 6: Row 4 -> Net-(D1-K)
- U1 pad 7: Row 5 -> Net-(D57-K)
Routing:
- net Net-(U1-GPIO9): track 114.3 -> 566.5 mm
- net Net-(U1-GPIO10): track 114.3 -> 530.6 mm
- net Net-(U1-GPIO14): track 0.00 -> 349.2 mm
- net Net-(U1-GPIO15): track 0.00 -> 338.1 mm
- net Net-(D33-K): track 0.00 -> 334.4 mm
- net Net-(D57-K): track 0.00 -> 328.8 mm
- net Net-(D41-K): track 0.00 -> 323.6 mm
- net Net-(U1-GPIO12): track 205.3 -> 480.9 mm
- net Row 4: track 228.6 -> 0.00 mm
- net Net-(D25-K): track 0.00 -> 220.7 mm
- net Net-(U1-GPIO13): track 205.9 -> 415.5 mm
- net Net-(D49-K): track 159.9 -> 357.0 mm
- net Net-(D10-K): track 0.00 -> 188.8 mm
- net Net-(U1-GPIO11): track 323.2 -> 504.6 mm
- net Net-(D1-K): track 0.00 -> 171.6 mm
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
Commit message: + update pcb
Parts:
- added REF**: Stabilizer_Cherry_MX_6.00u, PCM_Mounting_Keyboard_Stabilizer:Stabilizer_Cherry_MX_6.00u, F.Cu at (220.3, 202.0)
- added REF**: Stabilizer_Cherry_MX_2.00u, PCM_Mounting_Keyboard_Stabilizer:Stabilizer_Cherry_MX_2.00u, F.Cu at (334.6, 183.0)
- added SSD1331_SPI1: ~, OLED_Display_SSD1331_SPI:OLED_Display_SSD1331_SPI, F.Cu at (359.4, 95.3)
- added SW65: RotaryEncoder_Switch, Rotary_Encoder:RotaryEncoder_Alps_EC11E-Switch_Vertical_H20mm, F.Cu at (325.3, 96.8)
- moved D33 127.4 mm to (171.9, 102.0), turned to -90 degrees
- moved D34 123.1 mm to (184.4, 102.0), turned to -90 degrees
- moved D35 118.9 mm to (196.9, 102.0), turned to -90 degrees
- moved D25 114.2 mm to (169.4, 99.0), turned to -90 degrees
- moved D26 109.5 mm to (181.9, 99.0), turned to -90 degrees
- moved D40 108.7 mm to (259.4, 102.0), turned to -90 degrees
- moved D39 105.5 mm to (246.9, 102.0), turned to -90 degrees
- moved D27 105.0 mm to (194.4, 99.0), turned to -90 degrees
- moved D38 102.7 mm to (234.4, 102.0), turned to -90 degrees
- moved D17 102.0 mm to (166.9, 96.0), turned to -90 degrees
- moved D28 100.8 mm to (206.9, 99.0), turned to -90 degrees
- moved D37 100.2 mm to (221.9, 102.0), turned to -90 degrees
- moved D48 97.8 mm to (319.4, 99.0), turned to -90 degrees
- moved D18 96.9 mm to (179.4, 96.0), turned to -90 degrees
- moved D29 96.7 mm to (219.4, 99.0), turned to -90 degrees
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Connections:
- D1 pad 1: Net-(D1-K) -> Row 1
- D10 pad 1: Net-(D10-K) -> Row 2
- D11 pad 1: Net-(D10-K) -> Row 2
- D12 pad 1: Net-(D10-K) -> Row 2
- D13 pad 1: Net-(D10-K) -> Row 2
- D14 pad 1: Net-(D10-K) -> Row 2
- D15 pad 1: Net-(D10-K) -> Row 2
- D16 pad 1: Net-(D10-K) -> Row 2
- D17 pad 1: Net-(D17-K) -> Row 3
- D18 pad 1: Net-(D17-K) -> Row 3
- D19 pad 1: Net-(D17-K) -> Row 3
- D2 pad 1: Net-(D1-K) -> Row 1
- D20 pad 1: Net-(D17-K) -> Row 3
- D21 pad 1: Net-(D17-K) -> Row 3
- D22 pad 1: Net-(D17-K) -> Row 3
- D23 pad 1: Net-(D17-K) -> Row 3
- D24 pad 1: Net-(D17-K) -> Row 3
- D25 pad 1: Net-(D25-K) -> Row 4
- D26 pad 1: Net-(D25-K) -> Row 4
- D27 pad 1: Net-(D25-K) -> Row 4
- D28 pad 1: Net-(D25-K) -> Row 4
- D29 pad 1: Net-(D25-K) -> Row 4
- D3 pad 1: Net-(D1-K) -> Row 1
- D30 pad 1: Net-(D25-K) -> Row 4
- D31 pad 1: Net-(D25-K) -> Row 4
- D32 pad 1: Net-(D25-K) -> Row 4
- D33 pad 1: Net-(D33-K) -> Row 5
- D34 pad 1: Net-(D33-K) -> Row 5
- D35 pad 1: Net-(D33-K) -> Row 5
- D36 pad 1: Net-(D33-K) -> Row 5
- D37 pad 1: Net-(D33-K) -> Row 5
- D38 pad 1: Net-(D33-K) -> Row 5
- D39 pad 1: Net-(D33-K) -> Row 5
- D4 pad 1: Net-(D1-K) -> Row 1
- D40 pad 1: Net-(D33-K) -> Row 5
- D41 pad 1: Net-(D41-K) -> Row 6
- D42 pad 1: Net-(D41-K) -> Row 6
- D43 pad 1: Net-(D41-K) -> Row 6
- D44 pad 1: Net-(D41-K) -> Row 6
- D45 pad 1: Net-(D41-K) -> Row 6
- D46 pad 1: Net-(D41-K) -> Row 6
- D47 pad 1: Net-(D41-K) -> Row 6
- D48 pad 1: Net-(D41-K) -> Row 6
- D49 pad 1: Net-(D49-K) -> Row 7
- D5 pad 1: Net-(D1-K) -> Row 1
- D50 pad 1: Net-(D49-K) -> Row 7
- D51 pad 1: Net-(D49-K) -> Row 7
- D52 pad 1: Net-(D49-K) -> Row 7
- D53 pad 1: Net-(D49-K) -> Row 7
- D54 pad 1: Net-(D49-K) -> Row 7
- D55 pad 1: Net-(D49-K) -> Row 7
- D56 pad 1: Net-(D49-K) -> Row 7
- D57 pad 1: Net-(D57-K) -> Row 8
- D58 pad 1: Net-(D57-K) -> Row 8
- D59 pad 1: Net-(D57-K) -> Row 8
- D6 pad 1: Net-(D1-K) -> Row 1
- D60 pad 1: Net-(D57-K) -> Row 8
- D61 pad 1: Net-(D57-K) -> Row 8
- D62 pad 1: Net-(D57-K) -> Row 8
- D63 pad 1: Net-(D57-K) -> Row 8
- D64 pad 1: Net-(D57-K) -> Row 8
- D7 pad 1: Net-(D1-K) -> Row 1
- D8 pad 1: Net-(D1-K) -> Row 1
- D9 pad 1: Net-(D10-K) -> Row 2
- SW1 pad 2: Net-(U1-GPIO8) -> Col 1
- SW10 pad 2: Net-(U1-GPIO9) -> Col 2
- SW11 pad 2: Net-(U1-GPIO10) -> Col 3
- SW12 pad 2: Net-(U1-GPIO11) -> Col 4
- SW13 pad 2: Net-(U1-GPIO12) -> Col 5
- SW14 pad 2: Net-(U1-GPIO13) -> Col 6
- SW15 pad 2: Net-(U1-GPIO14) -> Col 7
- SW16 pad 2: Net-(U1-GPIO15) -> Col 8
- SW17 pad 2: Net-(U1-GPIO8) -> Col 1
- SW18 pad 2: Net-(U1-GPIO9) -> Col 2
- SW19 pad 2: Net-(U1-GPIO10) -> Col 3
- SW2 pad 2: Net-(U1-GPIO9) -> Col 2
- SW20 pad 2: Net-(U1-GPIO11) -> Col 4
- SW21 pad 2: Net-(U1-GPIO12) -> Col 5
- SW22 pad 2: Net-(U1-GPIO13) -> Col 6
- SW23 pad 2: Net-(U1-GPIO14) -> Col 7
- SW24 pad 2: Net-(U1-GPIO15) -> Col 8
- SW25 pad 2: Net-(U1-GPIO8) -> Col 1
- SW26 pad 2: Net-(U1-GPIO9) -> Col 2
- SW27 pad 2: Net-(U1-GPIO10) -> Col 3
- SW28 pad 2: Net-(U1-GPIO11) -> Col 4
- SW29 pad 2: Net-(U1-GPIO12) -> Col 5
- SW3 pad 2: Net-(U1-GPIO10) -> Col 3
- SW30 pad 2: Net-(U1-GPIO13) -> Col 6
- SW31 pad 2: Net-(U1-GPIO14) -> Col 7
- SW32 pad 2: Net-(U1-GPIO15) -> Col 8
- SW33 pad 2: Net-(U1-GPIO8) -> Col 1
- SW34 pad 2: Net-(U1-GPIO9) -> Col 2
- SW35 pad 2: Net-(U1-GPIO10) -> Col 3
- SW36 pad 2: Net-(U1-GPIO11) -> Col 4
- SW37 pad 2: Net-(U1-GPIO12) -> Col 5
- SW38 pad 2: Net-(U1-GPIO13) -> Col 6
- SW39 pad 2: Net-(U1-GPIO14) -> Col 7
- SW4 pad 2: Net-(U1-GPIO11) -> Col 4
- SW40 pad 2: Net-(U1-GPIO15) -> Col 8
- SW41 pad 2: Net-(U1-GPIO8) -> Col 1
- SW42 pad 2: Net-(U1-GPIO9) -> Col 2
- SW43 pad 2: Net-(U1-GPIO10) -> Col 3
- SW44 pad 2: Net-(U1-GPIO11) -> Col 4
- SW45 pad 2: Net-(U1-GPIO12) -> Col 5
- SW46 pad 2: Net-(U1-GPIO13) -> Col 6
- SW47 pad 2: Net-(U1-GPIO14) -> Col 7
- SW48 pad 2: Net-(U1-GPIO15) -> Col 8
- SW49 pad 2: Net-(U1-GPIO8) -> Col 1
- SW5 pad 2: Net-(U1-GPIO12) -> Col 5
- SW50 pad 2: Net-(U1-GPIO9) -> Col 2
- SW51 pad 2: Net-(U1-GPIO10) -> Col 3
- SW52 pad 2: Net-(U1-GPIO11) -> Col 4
- SW53 pad 2: Net-(U1-GPIO12) -> Col 5
- SW54 pad 2: Net-(U1-GPIO13) -> Col 6
- SW55 pad 2: Net-(U1-GPIO14) -> Col 7
- SW56 pad 2: Net-(U1-GPIO15) -> Col 8
- SW57 pad 2: Net-(U1-GPIO8) -> Col 1
- SW58 pad 2: Net-(U1-GPIO9) -> Col 2
- SW59 pad 2: Net-(U1-GPIO10) -> Col 3
- SW6 pad 2: Net-(U1-GPIO13) -> Col 6
- SW60 pad 2: Net-(U1-GPIO11) -> Col 4
- SW61 pad 2: Net-(U1-GPIO12) -> Col 5
- SW62 pad 2: Net-(U1-GPIO13) -> Col 6
- SW63 pad 2: Net-(U1-GPIO14) -> Col 7
- SW64 pad 2: Net-(U1-GPIO15) -> Col 8
- SW7 pad 2: Net-(U1-GPIO14) -> Col 7
- SW8 pad 2: Net-(U1-GPIO15) -> Col 8
- SW9 pad 2: Net-(U1-GPIO8) -> Col 1
- U1 pad 1: Net-(D33-K) -> Col 1
- U1 pad 10: Net-(D41-K) -> Col 8
- U1 pad 11: Net-(U1-GPIO8) -> Row 1
- U1 pad 12: Net-(U1-GPIO9) -> Row 2
- U1 pad 14: Net-(U1-GPIO10) -> Row 3
- U1 pad 15: Net-(U1-GPIO11) -> Row 4
- U1 pad 16: Net-(U1-GPIO12) -> Row 5
- U1 pad 17: Net-(U1-GPIO13) -> Row 6
- U1 pad 19: Net-(U1-GPIO14) -> Row 7
- U1 pad 2: Net-(D25-K) -> Col 2
- U1 pad 20: Net-(U1-GPIO15) -> Row 8
- U1 pad 21: unconnected-(U1-GPIO16-Pad21) -> Net-(SSD1331_SPI1-RES)
- U1 pad 22: unconnected-(U1-GPIO17-Pad22) -> Net-(SSD1331_SPI1-CS)
- U1 pad 24: unconnected-(U1-GPIO18-Pad24) -> Net-(SSD1331_SPI1-SCL)
- U1 pad 25: unconnected-(U1-GPIO19-Pad25) -> Net-(SSD1331_SPI1-SDA)
- U1 pad 26: unconnected-(U1-GPIO20-Pad26) -> Net-(SSD1331_SPI1-DC)
- U1 pad 31: unconnected-(U1-GPIO26_ADC0-Pad31) -> Net-(U1-GPIO26_ADC0)
- U1 pad 32: unconnected-(U1-GPIO27_ADC1-Pad32) -> Net-(U1-GPIO27_ADC1)
- U1 pad 34: unconnected-(U1-GPIO28_ADC2-Pad34) -> Net-(U1-GPIO28_ADC2)
- U1 pad 38: unconnected-(U1-GND-Pad38) -> GND
- U1 pad 4: Net-(D17-K) -> Col 3
- U1 pad 40: unconnected-(U1-VBUS-Pad40) -> VBUS
- U1 pad 5: Net-(D10-K) -> Col 4
- U1 pad 6: Net-(D1-K) -> Col 5
- U1 pad 7: Net-(D57-K) -> Col 6
- U1 pad 9: Net-(D49-K) -> Col 7
Routing:
- net Col 1: track 0.00 -> 595.8 mm
- net Col 2: track 0.00 -> 574.7 mm
- net Net-(U1-GPIO9): track 566.5 -> 0.00 mm
- net Col 3: track 0.00 -> 549.6 mm
- net Net-(U1-GPIO10): track 530.6 -> 0.00 mm
- net Col 4: track 0.00 -> 521.1 mm
- net Net-(U1-GPIO11): track 504.6 -> 0.00 mm
- net Col 5: track 0.00 -> 499.3 mm
- net Net-(U1-GPIO12): track 480.9 -> 0.00 mm
- net Col 6: track 0.00 -> 463.0 mm
- net Net-(U1-GPIO13): track 415.5 -> 0.00 mm
- net Col 8: track 0.00 -> 363.0 mm
- net Net-(D49-K): track 357.0 -> 0.00 mm
- net Col 7: track 0.00 -> 350.1 mm
- net Net-(U1-GPIO14): track 349.2 -> 0.00 mm
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
Commit message: + update pcb
Routing:
- net Net-(U1-GPIO28_ADC2): track 10.1 -> 0.00 mm
- net Net-(D38-A): track 179.8 -> 182.9 mm
- net Net-(D37-A): track 185.7 -> 188.8 mm
- net Net-(D39-A): track 175.4 -> 178.3 mm
- net Net-(D2-A): track 62.3 -> 64.8 mm
- net Net-(D17-A): track 104.7 -> 106.7 mm
- net Net-(D1-A): track 68.6 -> 70.6 mm
- net Net-(D9-A): track 88.0 -> 90.0 mm
- net Net-(D6-A): track 36.7 -> 38.7 mm
- net Net-(D5-A): track 43.3 -> 45.3 mm
- net Col 8: track 363.0 -> 361.5 mm
- net Net-(D4-A): track 48.6 -> 50.1 mm
- net Net-(D35-A): track 129.7 -> 128.4 mm
- net Net-(D3-A): track 57.0 -> 58.3 mm
- net Net-(D19-A): track 93.9 -> 92.9 mm
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
Commit message: + update pcb and schematic (add led)
Parts:
- added D65: LED, LED_THT:LED_D5.0mm, F.Cu at (317.3, 89.8)
- added R1: R, Resistor_THT:R_Axial_DIN0207_L6.3mm_D2.5mm_P10.16mm_Horizontal, F.Cu at (300.0, 81.3)
- moved D41 85.8 mm to (176.5, 98.1)
- moved D49 85.7 mm to (179.0, 100.1)
- moved D57 85.7 mm to (181.5, 102.1)
- moved D42 77.9 mm to (194.5, 98.1)
- moved D50 77.8 mm to (197.0, 100.1)
- moved D58 77.7 mm to (199.5, 102.1)
- moved D43 69.9 mm to (212.5, 98.1)
- moved D51 69.8 mm to (215.0, 100.1)
- moved D59 69.7 mm to (217.5, 102.1)
- moved D44 62.0 mm to (230.5, 98.1)
- moved D52 61.9 mm to (233.0, 100.1)
- moved D60 61.7 mm to (235.5, 102.1)
- moved D45 54.1 mm to (248.5, 98.1)
- moved D53 53.9 mm to (251.0, 100.1)
- moved D61 53.8 mm to (253.5, 102.1)
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Connections:
- U1 pad 27: unconnected-(U1-GPIO21-Pad27) -> Net-(U1-GPIO21)
Routing:
- net Net-(D47-A): track 118.9 -> 227.5 mm, vias 0 -> 1
- net Net-(D49-A): track 43.9 -> 133.9 mm
- net Net-(D50-A): track 47.5 -> 126.4 mm
- net Net-(D52-A): track 69.7 -> 141.7 mm
- net Net-(D57-A): track 72.4 -> 144.2 mm
- net Net-(D41-A): track 26.9 -> 98.0 mm
- net Net-(D42-A): track 30.7 -> 100.8 mm
- net Net-(D58-A): track 81.1 -> 150.0 mm
- net Net-(D51-A): track 59.3 -> 125.9 mm
- net Net-(D43-A): track 35.7 -> 101.3 mm
- net Net-(D59-A): track 89.9 -> 150.6 mm
- net Net-(D60-A): track 100.0 -> 159.1 mm
- net Row 6: track 216.5 -> 159.6 mm
- net Net-(D44-A): track 45.7 -> 102.1 mm
- net Col 6: track 463.0 -> 412.5 mm
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
Commit message: update pcb (remove one led and ssd1331 spi)
Parts:
- removed SSD1331_SPI1: ~, OLED_Display_SSD1331_SPI:OLED_Display_SSD1331_SPI
- added D66: LED, LED_THT:LED_D5.0mm, F.Cu at (345.6, 110.2)
- added H1: MountingHole, MountingHole:MountingHole_2.2mm_M2_Pad, F.Cu at (110.2, 90.2)
- added H10: MountingHole, MountingHole:MountingHole_2.2mm_M2_Pad, F.Cu at (239.4, 202.0)
- added H11: MountingHole, MountingHole:MountingHole_2.2mm_M2_Pad, F.Cu at (353.7, 192.5)
- added H2: MountingHole, MountingHole:MountingHole_2.2mm_M2_Pad, F.Cu at (369.1, 90.5)
- added H3: MountingHole, MountingHole:MountingHole_2.2mm_M2_Pad, F.Cu at (298.4, 92.8)
- added H4: MountingHole, MountingHole:MountingHole_2.2mm_M2_Pad, F.Cu at (110.2, 110.0)
- added H5: MountingHole, MountingHole:MountingHole_2.2mm_M2_Pad, F.Cu at (371.8, 108.7)
- added H6: MountingHole, MountingHole:MountingHole_2.2mm_M2_Pad, F.Cu at (125.1, 135.4)
- added H7: MountingHole, MountingHole:MountingHole_2.2mm_M2_Pad, F.Cu at (239.4, 135.4)
- added H8: MountingHole, MountingHole:MountingHole_2.2mm_M2_Pad, F.Cu at (353.7, 135.4)
- added H9: MountingHole, MountingHole:MountingHole_2.2mm_M2_Pad, F.Cu at (125.1, 192.5)
- added R2: R, Resistor_THT:R_Axial_DIN0207_L6.3mm_D2.5mm_P10.16mm_Horizontal, F.Cu at (337.7, 92.2)
- SW55: footprint PCM_Switch_Keyboard_Cherry_MX:SW_Cherry_MX_PCB_1.00u -> PCM_Switch_Keyboard_Cherry_MX:SW_Cherry_MX_PCB_2.00u
- SW56: footprint PCM_Switch_Keyboard_Cherry_MX:SW_Cherry_MX_PCB_2.00u -> PCM_Switch_Keyboard_Cherry_MX:SW_Cherry_MX_PCB_1.00u
- moved SW65 25.8 mm to (351.1, 98.4)
- moved R1 22.7 mm to (319.9, 92.2)
- moved D65 21.0 mm to (322.1, 110.2), turned to -90 degrees
- moved REF** 19.0 mm to (315.6, 183.0)
- moved D39 14.7 mm to (268.1, 91.0)
- moved D1 14.5 mm to (178.2, 91.0)
- moved D17 14.5 mm to (183.2, 95.0)
- moved D25 14.5 mm to (185.7, 97.0)
- moved D33 14.5 mm to (188.2, 99.0)
- moved D41 14.5 mm to (190.7, 101.0)
- moved D49 14.5 mm to (193.2, 103.0)
- moved D57 14.5 mm to (195.7, 105.0)
- moved D9 14.5 mm to (180.7, 93.0)
- moved D7 12.5 mm to (278.1, 99.0)
- moved D10 11.5 mm to (195.7, 93.0)
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Connections:
- U1 pad 21: Net-(SSD1331_SPI1-RES) -> unconnected-(U1-GPIO16-Pad21)
- U1 pad 22: Net-(SSD1331_SPI1-CS) -> unconnected-(U1-GPIO17-Pad22)
- U1 pad 24: Net-(SSD1331_SPI1-SCL) -> unconnected-(U1-GPIO18-Pad24)
- U1 pad 25: Net-(SSD1331_SPI1-SDA) -> unconnected-(U1-GPIO19-Pad25)
- U1 pad 26: Net-(SSD1331_SPI1-DC) -> unconnected-(U1-GPIO20-Pad26)
- U1 pad 29: unconnected-(U1-GPIO22-Pad29) -> Net-(U1-GPIO22)
Routing:
- net Net-(D47-A): track 227.5 -> 0.34 mm, vias 1 -> 0
- net Col 2: track 558.3 -> 361.8 mm, vias 1 -> 0
- net Col 3: track 539.6 -> 349.5 mm
- net Col 4: track 505.7 -> 321.2 mm
- net Col 5: track 483.3 -> 306.7 mm
- net Row 1: track 167.9 -> 0.00 mm
- net Row 2: track 164.7 -> 0.00 mm
- net Row 5: track 160.9 -> 0.57 mm
- net Row 6: track 159.6 -> 0.00 mm
- net Row 3: track 159.1 -> 0.00 mm
- net Row 7: track 157.8 -> 0.00 mm
- net Row 4: track 156.5 -> 0.00 mm
- net Row 8: track 155.6 -> 0.00 mm
- net Net-(D57-A): track 144.2 -> 0.34 mm
- net Net-(D48-A): track 141.9 -> 0.34 mm
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