File: pcb/KB426/KB426.kicad_pcb (KiCad board)
At the start: 2 copper layers, 147 parts, among them SW1 SW_Push_45deg, SW10 SW_Push_45deg, SW11 SW_Push_45deg, SW12 SW_Push_45deg, SW13 SW_Push_45deg, SW14 SW_Push_45deg, SW15 SW_Push_45deg, SW16 SW_Push_45deg, SW17 SW_Push_45deg, SW18 SW_Push_45deg, SW19 SW_Push_45deg, SW2 SW_Push_45deg, SW20 SW_Push_45deg, SW21 SW_Push_45deg, SW22 SW_Push_45deg, SW23 SW_Push_45deg, SW24 SW_Push_45deg, SW25 SW_Push_45deg, SW26 SW_Push_45deg, SW27 SW_Push_45deg, SW28 SW_Push_45deg, SW29 SW_Push_45deg, SW3 SW_Push_45deg, SW30 SW_Push_45deg, SW31 SW_Push_45deg, SW32 SW_Push_45deg, SW33 SW_Push_45deg, SW34 SW_Push_45deg, SW35 SW_Push_45deg, SW36 SW_Push_45deg, SW37 SW_Push_45deg, SW38 SW_Push_45deg, SW39 SW_Push_45deg, SW4 SW_Push_45deg, SW40 SW_Push_45deg, SW41 SW_Push_45deg, SW42 SW_Push_45deg, SW43 SW_Push_45deg, SW44 SW_Push_45deg, SW45 SW_Push_45deg, SW46 SW_Push_45deg, SW47 SW_Push_45deg, SW48 SW_Push_45deg, SW49 SW_Push_45deg, SW5 SW_Push_45deg, SW50 SW_Push_45deg, SW51 SW_Push_45deg, SW52 SW_Push_45deg, SW53 SW_Push_45deg, SW54 SW_Push_45deg, SW55 SW_Push_45deg, SW56 SW_Push_45deg, SW57 SW_Push_45deg, SW58 SW_Push_45deg, SW59 SW_Push_45deg, SW6 SW_Push_45deg, SW60 SW_Push_45deg, SW61 SW_Push_45deg, SW62 SW_Push_45deg, SW63 SW_Push_45deg, SW64 SW_Push_45deg, SW65 RotaryEncoder_Switch, SW7 SW_Push_45deg, SW8 SW_Push_45deg, SW9 SW_Push_45deg, U1 Pico

Commit message: + update pcb (redo all the layout)
Parts:
- removed R2: R, Resistor_THT:R_Axial_DIN0207_L6.3mm_D2.5mm_P10.16mm_Horizontal
- removed the SW47 at (363.2, 183.0)
- added D65: 1N4148, Diode_THT:D_DO-35_SOD27_P7.62mm_Horizontal, F.Cu at (246.0, 103.0)
- added D67: 1N4148, Diode_THT:D_DO-35_SOD27_P7.62mm_Horizontal, F.Cu at (262.0, 103.0)
- added D68: 1N4148, Diode_THT:D_DO-35_SOD27_P7.62mm_Horizontal, F.Cu at (262.0, 93.0)
- added D69: 1N4148, Diode_THT:D_DO-35_SOD27_P7.62mm_Horizontal, F.Cu at (278.0, 103.0)
- added D70: 1N4148, Diode_THT:D_DO-35_SOD27_P7.62mm_Horizontal, F.Cu at (278.0, 93.0)
- added D71: 1N4148, Diode_THT:D_DO-35_SOD27_P7.62mm_Horizontal, F.Cu at (294.0, 103.0)
- added D72: 1N4148, Diode_THT:D_DO-35_SOD27_P7.62mm_Horizontal, F.Cu at (294.0, 93.0)
- added ST7735S_80x160_SPI1: ~, SPI_Displays:ST7735S_80x160_SPI, F.Cu at (393.4, 99.9)
- added SW65: SW_Push_45deg, PCM_Switch_Keyboard_Cherry_MX:SW_Cherry_MX_PCB_1.00u, F.Cu at (268.0, 183.0)
- added SW66: SW_Push_45deg, PCM_Switch_Keyboard_Cherry_MX:SW_Cherry_MX_PCB_1.00u, F.Cu at (287.0, 183.0)
- added SW67: SW_Push_45deg, PCM_Switch_Keyboard_Cherry_MX:SW_Cherry_MX_PCB_1.00u, F.Cu at (306.1, 183.0)
- added SW68: SW_Push_45deg, PCM_Switch_Keyboard_Cherry_MX:SW_Cherry_MX_PCB_1.00u, F.Cu at (325.1, 183.0)
- added SW69: SW_Push_45deg, PCM_Switch_Keyboard_Cherry_MX:SW_Cherry_MX_PCB_2.00u, F.Cu at (353.7, 183.0)
- added SW70: SW_Push_45deg, PCM_Switch_Keyboard_Cherry_MX:SW_Cherry_MX_PCB_1.00u, F.Cu at (382.3, 183.0)
- added SW71: SW_Push_45deg, PCM_Switch_Keyboard_Cherry_MX:SW_Cherry_MX_PCB_1.00u, F.Cu at (401.3, 183.0)
- added SW72: SW_Push_45deg, PCM_Switch_Keyboard_Cherry_MX:SW_Cherry_MX_PCB_1.00u, F.Cu at (401.3, 202.0)
- added SW_RESET1: SW_Push, Button_Switch_THT:SW_PUSH_6mm, F.Cu at (371.4, 97.0)
- D66: value LED -> 1N4148; footprint LED_THT:LED_D5.0mm -> Diode_THT:D_DO-35_SOD27_P7.62mm_Horizontal
- SW46, SW62: footprint PCM_Switch_Keyboard_Cherry_MX:SW_Cherry_MX_PCB_1.00u -> PCM_Switch_Keyboard_Cherry_MX:SW_Cherry_MX_PCB_2.00u
- SW55: footprint PCM_Switch_Keyboard_Cherry_MX:SW_Cherry_MX_PCB_2.00u -> PCM_Switch_Keyboard_Cherry_MX:SW_Cherry_MX_PCB_1.00u
- moved SW63 134.7 mm to (401.3, 163.9)
- moved H6 116.8 mm to (236.8, 252.1)
- moved H2 115.7 mm to (411.7, 69.4)
- moved D66 101.1 mm to (246.0, 93.0), turned to -55 degrees
- moved SW64 97.1 mm to (382.3, 202.0)
- moved H11 87.1 mm to (456.2, 91.1)
- moved H4 85.2 mm to (457.1, 109.8)
- moved REF** 80.8 mm to (372.8, 125.8)
- moved SW55 76.8 mm to (382.3, 144.9)
- moved H7 72.9 mm to (426.6, 135.8)
- moved SW56 68.7 mm to (401.3, 144.9)
- moved D41 67.4 mm to (258.0, 103.0), turned to -55 degrees
- moved D40 67.3 mm to (226.0, 103.0), turned to -55 degrees
- moved D32 60.9 mm to (230.0, 103.0), turned to -55 degrees
- moved D49 60.9 mm to (254.0, 103.0), turned to -55 degrees
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- renumbered D65 to D100, H11 to H10, H2 to H11, H3 to H2, H4 to H3, H5 to H4, H6 to H5, H7 to H6, H8 to H7, H9 to H8, H10 to H9, SW65 to SW47
Connections:
- D66 pad 1: GND -> Row 9
- R1 pad 1: Net-(U1-GPIO21) -> Net-(U1-GPIO22)
- SW47 pad A: Net-(U1-GPIO28_ADC2) -> Rot CLK
- SW47 pad B: Net-(U1-GPIO27_ADC1) -> Rot DT
- SW47 pad S1: GND -> Col 7
- SW47 pad S2: Net-(U1-GPIO26_ADC0) -> Net-(D47-A)
- U1 pad 13: unconnected-(U1-GND-Pad13) -> GND
- U1 pad 18: unconnected-(U1-GND-Pad18) -> GND
- U1 pad 22: unconnected-(U1-GPIO17-Pad22) -> Net-(ST7735S_80x160_SPI1-CS)
- U1 pad 23: unconnected-(U1-GND-Pad23) -> GND
- U1 pad 24: unconnected-(U1-GPIO18-Pad24) -> Net-(ST7735S_80x160_SPI1-SCL)
- U1 pad 25: unconnected-(U1-GPIO19-Pad25) -> Net-(ST7735S_80x160_SPI1-SDA)
- U1 pad 26: unconnected-(U1-GPIO20-Pad26) -> Net-(ST7735S_80x160_SPI1-RES)
- U1 pad 27: Net-(U1-GPIO21) -> Net-(ST7735S_80x160_SPI1-DC)
- U1 pad 28: unconnected-(U1-GND-Pad28) -> GND
- U1 pad 3: unconnected-(U1-GND-Pad3) -> GND
- U1 pad 30: unconnected-(U1-RUN-Pad30) -> Net-(U1-RUN)
- U1 pad 31: Net-(U1-GPIO26_ADC0) -> unconnected-(U1-GPIO26_ADC0-Pad31)
- U1 pad 32: Net-(U1-GPIO27_ADC1) -> Rot CLK
- U1 pad 34: Net-(U1-GPIO28_ADC2) -> Rot DT
- U1 pad 36: unconnected-(U1-3V3-Pad36) -> 3V3
- U1 pad 8: unconnected-(U1-GND-Pad8) -> GND
Routing:
- net Net-(D64-A): track 0.34 -> 244.5 mm
- net Net-(D72-A): track 0.00 -> 217.2 mm
- net Col 1: track 477.4 -> 310.1 mm
- net Net-(D71-A): track 0.00 -> 164.3 mm
- net Net-(D70-A): track 0.00 -> 158.1 mm
- net Net-(D63-A): track 0.34 -> 145.6 mm
- net Net-(D69-A): track 0.00 -> 123.6 mm
- net Net-(D68-A): track 0.00 -> 123.3 mm
- net Col 5: track 306.7 -> 416.0 mm, vias 1 -> 0
- net Col 7: track 224.7 -> 330.1 mm
- net Net-(D55-A): track 0.00 -> 103.5 mm
- net Net-(D66-A): track 0.00 -> 102.9 mm
- net Net-(D41-A): track 117.3 -> 15.1 mm
- net Net-(D67-A): track 0.00 -> 100.1 mm
- net Net-(D62-A): track 40.7 -> 136.1 mm
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- added copper zone on B.Cu, net GND
Other:
- board outline added: 311.5 x 137 mm

Commit message: + update pcb (swap right tracks layer)
Parts:
- moved H4 399.3 mm to (58.1, 91.8)
- moved H11 399.2 mm to (57.9, 117.5)
- moved H7 382.8 mm to (45.2, 103.5)
- moved H2 377.4 mm to (34.9, 90.9)
- moved H10 330.5 mm to (45.0, 117.0)
- moved H6 253.6 mm to (32.7, 101.6)
- moved H8 140.0 mm to (57.8, 103.6)
- moved H5 79.3 mm to (21.8, 102.2)
- moved H1 74.1 mm to (22.1, 90.5)
- moved H3 34.3 mm to (46.5, 91.9)
Routing:
- net Net-(D48-A): track 0.00 -> 254.0 mm
- net Col 6: track 322.9 -> 435.1 mm
- net Col 8: track 176.8 -> 285.3 mm
- net Net-(D7-A): track 8.46 -> 38.9 mm
- net Net-(D15-A): track 30.9 -> 56.5 mm
- net Net-(D23-A): track 50.6 -> 71.7 mm
- net Col 7: track 330.1 -> 312.3 mm
- net Net-(D31-A): track 70.4 -> 87.7 mm
- net Net-(D40-A): track 170.4 -> 186.5 mm
- net Net-(D39-A): track 182.5 -> 197.7 mm
- net Net-(D32-A): track 61.2 -> 76.0 mm
- net Net-(D24-A): track 41.8 -> 55.3 mm
- net Net-(D16-A): track 22.9 -> 35.0 mm
- net Net-(D8-A): track 4.31 -> 14.9 mm
- net Col 2: track 310.4 -> 316.9 mm
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
Commit message: + update pcb
Parts:
- moved SW47 15.4 mm to (408.6, 128.3), turned to 180 degrees
- moved U1 1.00 mm to (132.1, 100.0)
Connections:
- SW47 pad S1: Col 7 -> Net-(D47-A)
- SW47 pad S2: Net-(D47-A) -> Col 7
Routing:
- net Col 8: track 285.3 -> 413.6 mm
- net Col 7: track 312.3 -> 439.6 mm
- net Row 7: track 0.00 -> 103.6 mm
- net Row 8: track 0.00 -> 103.5 mm
- net Col 6: track 435.1 -> 533.4 mm
- net Row 6: track 0.00 -> 96.4 mm
- net Row 9: track 0.00 -> 96.4 mm
- net Net-(D56-A): track 52.0 -> 141.3 mm
- net Col 5: track 420.4 -> 502.1 mm
- net Row 1: track 42.5 -> 116.7 mm
- net Row 2: track 42.4 -> 116.7 mm
- net Row 3: track 42.4 -> 109.6 mm
- net Col 4: track 357.6 -> 422.8 mm
- net Net-(D13-A): track 22.1 -> 75.3 mm
- net Net-(D5-A): track 0.34 -> 52.0 mm
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
Commit message: + update pcb, usb C hack
Parts:
- moved D100 22.6 mm to (344.7, 99.0), turned to 0 degrees
- moved R1 18.4 mm to (338.0, 90.1), turned to 0 degrees
Connections:
- SW47 pad A: Rot CLK -> Rot DT
- SW47 pad B: Rot DT -> Rot CLK
- U1 pad 21: unconnected-(U1-GPIO16-Pad21) -> Row 9
Routing:
- net Rot DT: track 0.00 -> 336.6 mm
- net Rot CLK: track 0.00 -> 326.9 mm
- net Net-(D17-A): track 126.7 -> 125.0 mm
- net Net-(D25-A): track 142.5 -> 141.8 mm
- net Net-(D33-A): track 158.2 -> 157.5 mm

Commit message: + update pcb (qwerty layout)
Parts:
- removed D69, D70, D71, D72: 1N4148, Diode_THT:D_DO-35_SOD27_P7.62mm_Horizontal
- removed SW69: SW_Push_45deg, PCM_Switch_Keyboard_Cherry_MX:SW_Cherry_MX_PCB_2.00u
- removed SW70, SW71, SW72: SW_Push_45deg, PCM_Switch_Keyboard_Cherry_MX:SW_Cherry_MX_PCB_1.00u
- added C1: 0.01 µf, Capacitor_SMD:C_1206_3216Metric_Pad1.33x1.80mm_HandSolder, F.Cu at (443.9, 84.9)
- added C2: 0.01 µf, Capacitor_SMD:C_1206_3216Metric_Pad1.33x1.80mm_HandSolder, F.Cu at (449.8, 84.6)
- added J1: Conn_01x03_Socket, Connector_PinHeader_2.54mm:PinHeader_1x03_P2.54mm_Vertical, F.Cu at (166.3, 91.1)
- added R1: 10k, Resistor_THT:R_Axial_DIN0207_L6.3mm_D2.5mm_P10.16mm_Horizontal, F.Cu at (458.4, 95.2)
- added R2: 10k, Resistor_THT:R_Axial_DIN0207_L6.3mm_D2.5mm_P10.16mm_Horizontal, F.Cu at (93.1, 93.8)
- added R3: 10k, Resistor_THT:R_Axial_DIN0207_L6.3mm_D2.5mm_P10.16mm_Horizontal, F.Cu at (444.1, 110.8)
- added R4: 10k, Resistor_THT:R_Axial_DIN0207_L6.3mm_D2.5mm_P10.16mm_Horizontal, F.Cu at (444.1, 114.8)
- added REF**: Stabilizer_Cherry_MX_2.00u, PCM_Mounting_Keyboard_Stabilizer:Stabilizer_Cherry_MX_2.00u, F.Cu at (370.4, 163.9)
- R5: renamed from R1; value R -> 390
- SW17, SW68: footprint PCM_Switch_Keyboard_Cherry_MX:SW_Cherry_MX_PCB_1.00u -> PCM_Switch_Keyboard_Cherry_MX:SW_Cherry_MX_PCB_1.75u
- SW25, SW61: footprint PCM_Switch_Keyboard_Cherry_MX:SW_Cherry_MX_PCB_1.00u -> PCM_Switch_Keyboard_Cherry_MX:SW_Cherry_MX_PCB_2.25u
- SW33, SW34, SW35: footprint PCM_Switch_Keyboard_Cherry_MX:SW_Cherry_MX_PCB_1.00u -> PCM_Switch_Keyboard_Cherry_MX:SW_Cherry_MX_PCB_1.25u
- SW36: footprint PCM_Switch_Keyboard_Cherry_MX:SW_Cherry_MX_PCB_6.00u -> PCM_Switch_Keyboard_Cherry_MX:SW_Cherry_MX_PCB_6.25u
- SW54, SW9: footprint PCM_Switch_Keyboard_Cherry_MX:SW_Cherry_MX_PCB_1.00u -> PCM_Switch_Keyboard_Cherry_MX:SW_Cherry_MX_PCB_1.50u
- SW62: footprint PCM_Switch_Keyboard_Cherry_MX:SW_Cherry_MX_PCB_2.00u -> PCM_Switch_Keyboard_Cherry_MX:SW_Cherry_MX_PCB_1.00u
- moved H2 372.2 mm to (407.1, 88.9)
- moved SW_RESET1 204.4 mm to (167.1, 101.1), turned to 0 degrees
- moved H1 86.6 mm to (108.6, 84.2)
- moved R5 75.5 mm to (403.9, 53.3), turned to -90 degrees
- moved D100 62.9 mm to (387.1, 52.5)
- moved D43 42.8 mm to (316.8, 103.0), turned to -45 degrees
- moved D44 42.8 mm to (316.8, 93.0), turned to -45 degrees
- moved D51 42.1 mm to (312.1, 103.0), turned to -45 degrees
- moved D52 42.1 mm to (312.1, 93.0), turned to -45 degrees
- moved D59 41.6 mm to (307.6, 103.0), turned to -45 degrees
- moved D60 41.6 mm to (307.6, 93.0), turned to -45 degrees
- moved D67 40.9 mm to (302.9, 103.0), turned to -45 degrees
- moved D68 40.9 mm to (302.9, 93.0), turned to -45 degrees
- moved D45 40.6 mm to (330.6, 103.0), turned to -45 degrees
- moved D46 40.6 mm to (330.6, 93.0), turned to -45 degrees
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Connections:
- net 3V3 renamed +3V3
- net VBUS renamed +5V
- D48 pad 1: Row 6 -> Row 8
- D64 pad 1: Row 8 -> Row 6
- SW47 pad A: Rot DT -> Net-(R2-Pad2)
- SW47 pad B: Rot CLK -> Net-(R1-Pad2)
- U1 pad 41: unconnected-(U1-SWCLK-Pad41) -> Net-(J1-Pin_3)
- U1 pad 42: unconnected-(U1-GND-Pad42) -> GND
- U1 pad 43: unconnected-(U1-SWDIO-Pad43) -> Net-(J1-Pin_1)
Routing:
- net Rot CLK: track 326.9 -> 49.2 mm
- net Net-(D72-A): track 208.2 -> 0.00 mm
- net Net-(D71-A): track 165.0 -> 0.00 mm
- net Net-(D70-A): track 160.0 -> 0.00 mm
- net Net-(D69-A): track 128.3 -> 0.00 mm
- net Col 6: track 533.4 -> 411.9 mm
- net Col 5: track 502.1 -> 385.8 mm
- net Net-(D64-A): track 233.4 -> 147.3 mm
- net Row 4: track 113.9 -> 34.6 mm
- net Row 7: track 103.6 -> 25.6 mm
- net Row 9: track 96.4 -> 20.9 mm
- net Row 8: track 103.5 -> 29.9 mm
- net Net-(D48-A): track 247.8 -> 176.3 mm
- net Row 1: track 116.7 -> 45.4 mm
- net Rot DT: track 336.6 -> 270.0 mm
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- added copper zone on F.Cu, net +3V3
Other:
- board size 311.5 x 137 mm -> 320.1 x 140.1 mm

Commit message: update pcb
Parts:
- moved H1 2.47 mm to (109.2, 86.6)
- moved U1 1.50 mm to (132.1, 101.5)
Other:
- board size 320.1 x 140.1 mm -> 310.3 x 134 mm
Changed lines of the file:
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@@
 	(footprint "MCU_RaspberryPi_and_Boards:RPi_Pico_SMD_TH"
 		(layer "F.Cu")
-		(at 132.06 100 90)
+		(at 132.06 101.5 90)
 		(descr "Through hole straight pin header, 2x20, 2.54mm pitch, double rows")
 		(tags "Through hole pin header THT 2x20 2.54mm double row")
@@
 	(footprint "MountingHole:MountingHole_2.2mm_M2_Pad"
 		(layer "F.Cu")
-		(at 108.56 84.19)
+		(at 109.2 86.575)
 		(descr "Mounting Hole 2.2mm, M2")
 		(tags "mounting hole 2.2mm m2")
@@
 	)
 	(gr_rect
-		(start 96.17 76.17)
+		(start 105.95 82.225)
 		(end 416.23 216.23)
 		(stroke

Commit message: update pcb
Parts:
- removed H11: MountingHole, MountingHole:MountingHole_2.2mm_M2_Pad
- removed J1: Conn_01x03_Socket, Connector_PinHeader_2.54mm:PinHeader_1x03_P2.54mm_Vertical
- removed ST7735S_80x160_SPI1: ~, SPI_Displays:ST7735S_80x160_SPI
- removed the SW48 at (382.3, 202.0)
- added D69: 1N4148, Diode_THT:D_DO-35_SOD27_P7.62mm_Horizontal, F.Cu at (333.5, 97.2)
- added D70: LED, LED_THT:LED_D5.0mm, F.Cu at (319.6, 92.7)
- added J3: Conn_01x06_Socket, Connector_PinHeader_2.54mm:PinHeader_2x03_P2.54mm_Vertical, F.Cu at (162.3, 95.2)
- added R5: 390, Resistor_THT:R_Axial_DIN0207_L6.3mm_D2.5mm_P10.16mm_Horizontal, F.Cu at (288.4, 93.4)
- added REF**: Stabilizer_Cherry_MX_2.00u, PCM_Mounting_Keyboard_Stabilizer:Stabilizer_Cherry_MX_2.00u, F.Cu at (370.4, 163.9)
- added SSD1306_128x32_i2c1: ~, SPI_Displays:SSD1306_128x32_i2c, F.Cu at (366.0, 101.0)
- added SW47: SW_Push_45deg, PCM_Switch_Keyboard_Cherry_MX:SW_Cherry_MX_PCB_1.00u, F.Cu at (401.3, 125.8)
- added SW69: SW_Push_45deg, PCM_Switch_Keyboard_Cherry_MX:SW_Cherry_MX_PCB_1.00u, F.Cu at (382.3, 202.0)
- C1, C2: footprint Capacitor_SMD:C_1206_3216Metric_Pad1.33x1.80mm_HandSolder -> Capacitor_THT:C_Disc_D3.0mm_W1.6mm_P2.50mm
- SW60: footprint PCM_Switch_Keyboard_Cherry_MX:SW_Cherry_MX_PCB_1.00u -> PCM_Switch_Keyboard_Cherry_MX:SW_Cherry_MX_PCB_2.25u
- SW61: footprint PCM_Switch_Keyboard_Cherry_MX:SW_Cherry_MX_PCB_2.25u -> PCM_Switch_Keyboard_Cherry_MX:SW_Cherry_MX_PCB_1.00u
- SW66: footprint PCM_Switch_Keyboard_Cherry_MX:SW_Cherry_MX_PCB_1.00u -> PCM_Switch_Keyboard_Cherry_MX:SW_Cherry_MX_PCB_1.75u
- SW68: footprint PCM_Switch_Keyboard_Cherry_MX:SW_Cherry_MX_PCB_1.75u -> PCM_Switch_Keyboard_Cherry_MX:SW_Cherry_MX_PCB_1.00u
- moved H5 380.9 mm to (391.8, 192.5)
- moved H7 346.1 mm to (389.4, 139.3)
- moved H6 324.8 mm to (351.5, 163.7)
- moved R2 280.6 mm to (373.3, 109.5), turned to 0 degrees
- moved REF** 243.6 mm to (127.5, 183.0)
- moved H4 204.9 mm to (258.4, 134.8)
- moved H10 151.3 mm to (191.8, 153.8)
- moved SW56 120.6 mm to (282.3, 163.9)
- moved H8 117.3 mm to (129.9, 202.0)
- moved R6 110.2 mm to (301.2, 93.4), turned to 0 degrees
- moved C2 99.6 mm to (353.3, 109.5), turned to 180 degrees
- moved C1 94.8 mm to (353.3, 113.0), turned to 180 degrees
- moved SW64 92.5 mm to (310.8, 183.0)
- moved SW63 90.5 mm to (291.8, 183.0)
- moved R1 86.9 mm to (373.3, 113.0), turned to 0 degrees
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- renumbered D100 to D71, R5 to R6, SW47 to SW48
Connections:
- D48 pad 1: Row 8 -> Row 6
- D56 pad 1: Row 7 -> Row 8
- D63 pad 1: Row 8 -> Row 9
- D64 pad 1: Row 6 -> Row 9
- SW48 pad S1: Net-(D47-A) -> Col 8
- SW48 pad S2: Col 7 -> Net-(D48-A)
- SW56 pad 2: Col 8 -> Col 1
- SW57 pad 2: Col 1 -> Col 2
- SW58 pad 2: Col 2 -> Col 3
- SW59 pad 2: Col 3 -> Col 4
- SW60 pad 2: Col 4 -> Col 5
- SW61 pad 2: Col 5 -> Col 6
- SW62 pad 2: Col 6 -> Col 7
- SW63 pad 2: Col 7 -> Col 1
- SW64 pad 2: Col 8 -> Col 2
- SW65 pad 2: Col 1 -> Col 3
- SW66 pad 2: Col 2 -> Col 4
- SW67 pad 2: Col 3 -> Col 5
- SW68 pad 2: Col 4 -> Col 6
- U1 pad 22: Net-(ST7735S_80x160_SPI1-CS) -> unconnected-(U1-GPIO17-Pad22)
- U1 pad 26: Net-(ST7735S_80x160_SPI1-RES) -> unconnected-(U1-GPIO20-Pad26)
- U1 pad 27: Net-(ST7735S_80x160_SPI1-DC) -> unconnected-(U1-GPIO21-Pad27)
Routing:
- net Rot DT: track 270.0 -> 5.00 mm
- net Net-(SSD1306_128x32_i2c1-SDA): track 16.8 -> 207.8 mm
- net Net-(SSD1306_128x32_i2c1-SCK): track 15.8 -> 205.9 mm
- net Row 7: track 25.6 -> 209.2 mm
- net Row 8: track 29.9 -> 203.4 mm
- net Net-(D69-A): track 0.00 -> 173.5 mm
- net Row 6: track 47.8 -> 220.9 mm
- net Net-(U1-GPIO22): track 0.00 -> 172.8 mm
- net Row 9: track 20.9 -> 181.5 mm
- net Row 1: track 45.4 -> 155.5 mm
- net Row 4: track 34.6 -> 139.5 mm
- net Net-(D48-A): track 176.3 -> 73.7 mm
- net Col 8: track 347.7 -> 422.8 mm
- net Col 1: track 343.0 -> 415.6 mm
- net Col 2: track 370.1 -> 437.5 mm
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- removed copper zone on F.Cu, net +3V3
- removed copper zone on B.Cu, net GND
Other:
- board size 310.3 x 134 mm -> 305 x 123.5 mm
- board text added: "CapsLock"
- board text added: "GND"
- board text added: "POWER"
- board text added: "RX"
- board text added: "SWCLK"
- board text added: "SWDIO"
- board text added: "TX"

Commit message: + update pcb
Parts:
- added J2: Conn_01x03_Socket, Connector_PinHeader_2.54mm:PinHeader_1x03_P2.54mm_Vertical, B.Cu at (170.7, 70.6)
- moved R5 11.6 mm to (276.8, 92.5)
- moved R6 11.5 mm to (289.8, 92.5)
- moved H1 9.16 mm to (164.2, 92.5)
- moved SW_RESET1 8.67 mm to (167.9, 112.0), turned to 180 degrees
- moved C2 5.02 mm to (358.3, 112.5)
- moved R2 5.02 mm to (363.3, 112.5)
- moved R4 5.02 mm to (378.3, 112.5)
- moved C1 5.00 mm to (358.3, 109.5)
- moved R1 5.00 mm to (363.3, 109.5)
- moved R3 5.00 mm to (378.3, 109.5)
- moved J1 4.69 mm to (165.0, 99.0), turned to 0 degrees
- moved SSD1306_128x32_i2c1 4.53 mm to (370.5, 100.9)
- moved D70 0.34 mm to (319.6, 93.0)
- moved D71 0.13 mm to (329.6, 93.0)
- renumbered C2 to C1, C1 to C2, J3 to J1, R4 to R1, R3 to R2, R2 to R3, R1 to R4
Connections:
- J1 pad 1: Net-(J3-Pin_1) -> Net-(J1-Pin_1)
- J1 pad 2: Col 2 -> Net-(J1-Pin_2)
- J1 pad 5: Net-(J3-Pin_5) -> Net-(J1-Pin_5)
- J1 pad 6: Col 1 -> Net-(J1-Pin_6)
- R6 pad 1: Net-(U1-GPIO22) -> Net-(U1-GPIO27_ADC1)
- U1 pad 21: Row 9 -> Net-(J1-Pin_6)
- U1 pad 22: unconnected-(U1-GPIO17-Pad22) -> Net-(J1-Pin_2)
- U1 pad 24: Net-(SSD1306_128x32_i2c1-SCK) -> Row 9
- U1 pad 25: Net-(SSD1306_128x32_i2c1-SDA) -> Net-(J2-Pin_2)
- U1 pad 26: unconnected-(U1-GPIO20-Pad26) -> Net-(SSD1306_128x32_i2c1-SDA)
- U1 pad 27: unconnected-(U1-GPIO21-Pad27) -> Net-(SSD1306_128x32_i2c1-SCK)
- U1 pad 29: Net-(U1-GPIO22) -> Rot DT
- U1 pad 31: unconnected-(U1-GPIO26_ADC0-Pad31) -> Rot CLK
- U1 pad 32: Rot CLK -> Net-(U1-GPIO27_ADC1)
- U1 pad 34: Rot DT -> unconnected-(U1-GPIO28_ADC2-Pad34)
- U1 pad 39: unconnected-(U1-VSYS-Pad39) -> +5V
- U1 pad 41: Net-(J3-Pin_1) -> Net-(J1-Pin_5)
- U1 pad 43: Net-(J3-Pin_5) -> Net-(J1-Pin_1)
Routing:
- net +3V3: track 0.00 -> 282.1 mm
- net Rot CLK: track 5.00 -> 251.6 mm
- net Rot DT: track 5.00 -> 244.4 mm
- net +5V: track 0.00 -> 238.5 mm
- net Net-(J2-Pin_2): track 0.00 -> 202.6 mm
- net Net-(U1-GPIO22): track 172.8 -> 0.00 mm
- net Net-(U1-GPIO27_ADC1): track 0.00 -> 165.8 mm, vias 0 -> 1
- net Col 1: track 415.6 -> 342.8 mm, vias 0 -> 1
- net Col 2: track 437.5 -> 377.9 mm, vias 0 -> 1
- net Net-(U1-RUN): track 0.00 -> 46.5 mm, vias 0 -> 1
- net Row 9: track 181.5 -> 216.1 mm, vias 0 -> 2
- net Net-(J1-Pin_6): track 0.00 -> 27.7 mm, vias 0 -> 1
- net Net-(J1-Pin_2): track 0.00 -> 25.2 mm, vias 0 -> 1
- net Col 8: track 422.8 -> 443.1 mm, vias 0 -> 1
- net GND: track 0.00 -> 15.5 mm
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- added copper zone on B.Cu, net GND
Other:
- board text removed: "SWCLK"
- board text removed: "SWDIO"
