File: pcb/KB426/KB426.kicad_pcb (KiCad board)
At the start: 2 copper layers, 305 x 123.5 mm, 167 parts, among them J1 Conn_01x06_Socket, J2 Conn_01x03_Socket, SW1 SW_Push_45deg, SW10 SW_Push_45deg, SW11 SW_Push_45deg, SW12 SW_Push_45deg, SW13 SW_Push_45deg, SW14 SW_Push_45deg, SW15 SW_Push_45deg, SW16 SW_Push_45deg, SW17 SW_Push_45deg, SW18 SW_Push_45deg, SW19 SW_Push_45deg, SW2 SW_Push_45deg, SW20 SW_Push_45deg, SW21 SW_Push_45deg, SW22 SW_Push_45deg, SW23 SW_Push_45deg, SW24 SW_Push_45deg, SW25 SW_Push_45deg, SW26 SW_Push_45deg, SW27 SW_Push_45deg, SW28 SW_Push_45deg, SW29 SW_Push_45deg, SW3 SW_Push_45deg, SW30 SW_Push_45deg, SW31 SW_Push_45deg, SW32 SW_Push_45deg, SW33 SW_Push_45deg, SW34 SW_Push_45deg, SW35 SW_Push_45deg, SW36 SW_Push_45deg, SW37 SW_Push_45deg, SW38 SW_Push_45deg, SW39 SW_Push_45deg, SW4 SW_Push_45deg, SW40 SW_Push_45deg, SW41 SW_Push_45deg, SW42 SW_Push_45deg, SW43 SW_Push_45deg, SW44 SW_Push_45deg, SW45 SW_Push_45deg, SW46 SW_Push_45deg, SW47 SW_Push_45deg, SW48 RotaryEncoder_Switch, SW49 SW_Push_45deg, SW5 SW_Push_45deg, SW50 SW_Push_45deg, SW51 SW_Push_45deg, SW52 SW_Push_45deg, SW53 SW_Push_45deg, SW54 SW_Push_45deg, SW55 SW_Push_45deg, SW56 SW_Push_45deg, SW57 SW_Push_45deg, SW58 SW_Push_45deg, SW59 SW_Push_45deg, SW6 SW_Push_45deg, SW60 SW_Push_45deg, SW61 SW_Push_45deg, SW62 SW_Push_45deg, SW63 SW_Push_45deg, SW64 SW_Push_45deg, SW65 SW_Push_45deg, SW66 SW_Push_45deg, SW67 SW_Push_45deg, SW68 SW_Push_45deg, SW69 SW_Push_45deg, SW7 SW_Push_45deg, SW8 SW_Push_45deg, SW9 SW_Push_45deg, U1 Pico

Commit message: pcb v1
Parts:
- removed D70, D71: LED, LED_THT:LED_D5.0mm
- removed J2: Conn_01x03_Socket, Connector_PinHeader_2.54mm:PinHeader_1x03_P2.54mm_Vertical
- added C10: 100nF, Capacitor_SMD:C_0603_1608Metric, B.Cu at (396.3, 190.9)
- added C11: 100nF, Capacitor_SMD:C_0603_1608Metric, B.Cu at (348.7, 190.9)
- added C12: 100nF, Capacitor_SMD:C_0603_1608Metric, B.Cu at (301.1, 190.9)
- added C13: 100nF, Capacitor_SMD:C_0603_1608Metric, B.Cu at (253.4, 190.9)
- added C14: 100nF, Capacitor_SMD:C_0603_1608Metric, B.Cu at (205.8, 190.9)
- added C15: 100nF, Capacitor_SMD:C_0603_1608Metric, B.Cu at (158.2, 190.9)
- added C16: 100nF, Capacitor_SMD:C_0603_1608Metric, B.Cu at (119.0, 190.9)
- added C17: 100nF, Capacitor_SMD:C_0603_1608Metric, B.Cu at (110.6, 152.6)
- added C18: 100nF, Capacitor_SMD:C_0603_1608Metric, B.Cu at (115.2, 102.4)
- added C3: 100nF, Capacitor_SMD:C_0603_1608Metric, B.Cu at (176.2, 94.6)
- added C4: 100nF, Capacitor_SMD:C_0603_1608Metric, B.Cu at (213.7, 94.6)
- added C5: 100nF, Capacitor_SMD:C_0603_1608Metric, B.Cu at (263.7, 94.6)
- added C6: 100nF, Capacitor_SMD:C_0603_1608Metric, B.Cu at (303.7, 94.6)
- added C7: 100nF, Capacitor_SMD:C_0603_1608Metric, B.Cu at (352.2, 99.9)
- added C8: 100nF, Capacitor_SMD:C_0603_1608Metric, B.Cu at (396.5, 108.4)
- added C9: 100nF, Capacitor_SMD:C_0603_1608Metric, B.Cu at (396.3, 152.6)
- added CAPSLOCK: LED, LED_THT:LED_D5.0mm, F.Cu at (339.8, 94.6)
- added D72: WS2812B, LED_SMD:LED_WS2812B_PLCC4_5.0x5.0mm_P3.2mm, B.Cu at (181.0, 95.0)
- added D73: WS2812B, LED_SMD:LED_WS2812B_PLCC4_5.0x5.0mm_P3.2mm, B.Cu at (218.5, 95.0)
- added D74: WS2812B, LED_SMD:LED_WS2812B_PLCC4_5.0x5.0mm_P3.2mm, B.Cu at (268.5, 95.0)
- added D75: WS2812B, LED_SMD:LED_WS2812B_PLCC4_5.0x5.0mm_P3.2mm, B.Cu at (308.5, 95.0)
- added D76: WS2812B, LED_SMD:LED_WS2812B_PLCC4_5.0x5.0mm_P3.2mm, B.Cu at (357.2, 99.0)
- added D77: WS2812B, LED_SMD:LED_WS2812B_PLCC4_5.0x5.0mm_P3.2mm, B.Cu at (401.3, 107.5)
- added D78: WS2812B, LED_SMD:LED_WS2812B_PLCC4_5.0x5.0mm_P3.2mm, B.Cu at (401.3, 151.7)
- added D79: WS2812B, LED_SMD:LED_WS2812B_PLCC4_5.0x5.0mm_P3.2mm, B.Cu at (401.3, 190.0)
- added D80: WS2812B, LED_SMD:LED_WS2812B_PLCC4_5.0x5.0mm_P3.2mm, B.Cu at (353.7, 190.0)
- added D81: WS2812B, LED_SMD:LED_WS2812B_PLCC4_5.0x5.0mm_P3.2mm, B.Cu at (306.1, 190.0)
- added D82: WS2812B, LED_SMD:LED_WS2812B_PLCC4_5.0x5.0mm_P3.2mm, B.Cu at (258.4, 190.0)
- added D83: WS2812B, LED_SMD:LED_WS2812B_PLCC4_5.0x5.0mm_P3.2mm, B.Cu at (210.8, 190.0)
- added D84: WS2812B, LED_SMD:LED_WS2812B_PLCC4_5.0x5.0mm_P3.2mm, B.Cu at (163.2, 190.0)
- added D85: WS2812B, LED_SMD:LED_WS2812B_PLCC4_5.0x5.0mm_P3.2mm, B.Cu at (124.0, 190.0)
- added D86: WS2812B, LED_SMD:LED_WS2812B_PLCC4_5.0x5.0mm_P3.2mm, B.Cu at (115.6, 151.7)
- added D87: WS2812B, LED_SMD:LED_WS2812B_PLCC4_5.0x5.0mm_P3.2mm, B.Cu at (120.2, 101.5)
- added POWER: LED, LED_THT:LED_D5.0mm, F.Cu at (329.8, 94.6)
- moved R5 81.8 mm to (356.9, 109.4), turned to 180 degrees
- moved R6 70.0 mm to (356.9, 112.4), turned to 180 degrees
- moved H7 5.54 mm to (389.4, 144.9)
- moved C2 4.80 mm to (362.0, 109.4), turned to -90 degrees
- moved SSD1306_128x32_i2c1 3.53 mm to (367.0, 101.0)
- moved R1 1.23 mm to (364.5, 109.4)
- moved R2 1.23 mm to (364.5, 112.4)
- moved C1 1.15 mm to (359.5, 109.4), turned to -90 degrees
- moved R3 1.08 mm to (377.2, 109.4)
- moved R4 1.08 mm to (377.2, 112.4)
- renumbered SW_RESET1 to RESET
Connections:
- net Net-(J1-Pin_1) renamed swdio
- net Net-(J1-Pin_5) renamed swclk
- J1 pad 2: Net-(J1-Pin_2) -> uart tx
- J1 pad 6: Net-(J1-Pin_6) -> uart rx
- U1 pad 21: Net-(J1-Pin_6) -> uart tx
- U1 pad 22: Net-(J1-Pin_2) -> uart rx
- U1 pad 25: Net-(J2-Pin_2) -> leds
Routing:
- net +5V: track 238.5 -> 1184.4 mm
- net Net-(J2-Pin_2): track 202.6 -> 0.00 mm
- net Net-(U1-GPIO27_ADC1): track 165.8 -> 242.6 mm, vias 1 -> 0
- net Col 5: track 421.2 -> 495.8 mm
- net Net-(D86-DOUT): track 0.00 -> 73.1 mm
- net Net-(D85-DOUT): track 0.00 -> 64.3 mm, vias 0 -> 2
- net Net-(D79-DOUT): track 0.00 -> 58.1 mm, vias 0 -> 2
- net Net-(D80-DOUT): track 0.00 -> 56.6 mm, vias 0 -> 2
- net Net-(D82-DOUT): track 0.00 -> 56.1 mm, vias 0 -> 2
- net Net-(D81-DOUT): track 0.00 -> 55.9 mm, vias 0 -> 2
- net Net-(D83-DOUT): track 0.00 -> 55.9 mm, vias 0 -> 2
- net Net-(D77-DOUT): track 0.00 -> 51.0 mm
- net Net-(D84-DOUT): track 0.00 -> 48.5 mm, vias 0 -> 2
- net Net-(D75-DOUT): track 0.00 -> 48.0 mm
- net Net-(D73-DOUT): track 0.00 -> 47.3 mm
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Other:
- board text removed: "CapsLock"
- board text removed: "POWER"

Commit message: little pcb fix
Routing:
- net +5V: track 1184.4 -> 1185.5 mm
Changed lines of the file:
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@@
 		(tags "Resistor Axial_DIN0207 series Axial Horizontal pin pitch 10.16mm 0.25W = 1/4W length 6.3mm diameter 2.5mm")
 		(property "Reference" "R5"
-			(at 5.08 -0.01 360)
+			(at 5.08 -0.01 0)
 			(layer "F.SilkS")
 			(effects
@@
 		)
 		(property "Value" "390"
-			(at 5.08 -0.03 360)
+			(at 5.08 -0.03 0)
 			(layer "F.Fab")
 			(effects
@@
 		)
 		(fp_text user "${REFERENCE}"
-			(at 5.08 0 360)
+			(at 5.08 0 0)
 			(layer "F.Fab")
 			(effects
@@
 		(tags "Resistor Axial_DIN0207 series Axial Horizontal pin pitch 10.16mm 0.25W = 1/4W length 6.3mm diameter 2.5mm")
 		(property "Reference" "R6"
-			(at 5.02 0 360)
+			(at 5.02 0 0)
 			(layer "F.SilkS")
 			(effects
@@
 		)
 		(property "Value" "390"
-			(at 5.08 0 360)
+			(at 5.08 0 0)
 			(layer "F.Fab")
 			(effects
@@
 		)
 		(fp_text user "${REFERENCE}"
-			(at 5.08 0 360)
+			(at 5.08 0 0)
 			(layer "F.Fab")
 			(effects
@@
 	)
 	(segment
+		(start 183.45 91.575)
+		(end 183.45 93.35)
+		(width 0.7)
+		(layer "B.Cu")
+		(net 107)
+	)
+	(segment
 		(start 301.94 194.03)
 		(end 309 194.03)
@@
 	)
 	(segment
+		(start 310.95 91.575)
+		(end 310.95 93.35)
+		(width 0.7)
+		(layer "B.Cu")
+		(net 107)
+	)
+	(segment
+		(start 180.925 89.05)
+		(end 183.45 91.575)
+		(width 0.7)
+		(layer "B.Cu")
+		(net 107)
+	)
+	(segment
 		(start 358.06 210.79)
 		(end 300.79 210.79)
@@
 	)
 	(segment
-		(start 310.95 91.7)
-		(end 310.95 93.35)
+		(start 270.95 91.575)
+		(end 270.95 93.35)
 		(width 0.7)
 		(layer "B.Cu")
@@
 	)
 	(segment
-		(start 192.48 205.87)
-		(end 197.4 210.79)
+		(start 217.84 89.05)
+		(end 180.35 89.05)
 		(width 0.7)
 		(layer "B.Cu")
@@
 	)
 	(segment
-		(start 183.45 93.35)
-		(end 182.45 94.35)
+		(start 192.48 205.87)
+		(end 197.4 210.79)
 		(width 0.7)
 		(layer "B.Cu")
@@
 	)
 	(segment
-		(start 354.97 89.05)
-		(end 407.85 89.05)
+		(start 183.45 93.35)
+		(end 182.45 94.35)
 		(width 0.7)
 		(layer "B.Cu")
@@
 	)
 	(segment
+		(start 407.85 89.05)
+		(end 410.08 91.28)
+		(width 0.7)
+		(layer "B.Cu")
+		(net 107)
+	)
+	(segment
 		(start 118.025 149.265)
 		(end 117.01 148.25)
@@
 	)
 	(segment
-		(start 108.73 89.05)
-		(end 181.34 89.05)
-		(width 0.7)
-		(layer "B.Cu")
-		(net 107)
-	)
-	(segment
 		(start 213.275 188.35)
 		(end 211.4 188.35)
@@
 	)
 	(segment
-		(start 406.39 103.58)
-		(end 406.39 104.83)
-		(width 0.7)
-		(layer "B.Cu")
-		(net 107)
-	)
-	(segment
-		(start 268.06 89.05)
-		(end 270.95 91.94)
+		(start 354.97 89.05)
+		(end 407.85 89.05)
 		(width 0.7)
 		(layer "B.Cu")
@@
 	)
 	(segment
-		(start 220.95 91.58)
-		(end 220.95 93.35)
+		(start 410.08 98.545)
+		(end 406.39 102.235)
 		(width 0.7)
 		(layer "B.Cu")
@@
 	)
 	(segment
-		(start 135.73 210.79)
-		(end 134.04 209.1)
-		(width 0.7)
-		(layer "B.Cu")
-		(net 107)
-	)
-	(segment
-		(start 307.63 89.05)
-		(end 308.3 89.05)
+		(start 220.95 91.58)
+		(end 220.95 93.35)
 		(width 0.7)
 		(layer "B.Cu")
@@
 	)
 	(segment
-		(start 183.46 91.17)
-		(end 183.45 91.18)
+		(start 135.73 210.79)
+		(end 134.04 209.1)
 		(width 0.7)
 		(layer "B.Cu")
@@
 	)
 	(segment
+		(start 180.35 89.05)
+		(end 180.925 89.05)
+		(width 0.7)
+		(layer "B.Cu")
+		(net 107)
+	)
+	(segment
 		(start 220.95 93.35)
 		(end 219.95 94.35)
@@
 	)
 	(segment
+		(start 410.08 91.28)
+		(end 410.08 98.545)
+		(width 0.7)
+		(layer "B.Cu")
+		(net 107)
+	)
+	(segment
 		(start 134.04 209.1)
 		(end 134.04 192.69)
@@
 	)
 	(segment
+		(start 268.06 89.05)
+		(end 268.425 89.05)
+		(width 0.7)
+		(layer "B.Cu")
+		(net 107)
+	)
+	(segment
 		(start 122.7 99.85)
 		(end 120.95 101.6)
@@
 	)
 	(segment
+		(start 307.63 89.05)
+		(end 308.425 89.05)
+		(width 0.7)
+		(layer "B.Cu")
+		(net 107)
+	)
+	(segment
 		(start 406.39 110.845962)
 		(end 410.08 114.535962)
@@
 	)
 	(segment
-		(start 181.34 89.05)
-		(end 217.84 89.05)
-		(width 0.7)
-		(layer "B.Cu")
-		(net 107)
-	)
-	(segment
 		(start 263.24 188.35)
 		(end 260.9 188.35)
@@
 	)
 	(segment
-		(start 308.3 89.05)
-		(end 310.95 91.7)
-		(width 0.7)
-		(layer "B.Cu")
-		(net 107)
-	)
-	(segment
 		(start 410.08 184.09)
 		(end 405.82 188.35)
@@
 	)
 	(segment
-		(start 181.34 89.05)
-		(end 183.46 91.17)
+		(start 180.35 89.05)
+		(end 108.73 89.05)
 		(width 0.7)
 		(layer "B.Cu")
@@
 	)
 	(segment
-		(start 168.2 188.35)
-		(end 173.88 194.03)
+		(start 268.425 89.05)
+		(end 270.95 91.575)
 		(width 0.7)
 		(layer "B.Cu")
@@
 	)
 	(segment
-		(start 183.45 91.18)
-		(end 183.45 93.35)
+		(start 168.2 188.35)
+		(end 173.88 194.03)
 		(width 0.7)
 		(layer "B.Cu")
@@
 	)
 	(segment
-		(start 403.7748 105.85)
-		(end 405.37 105.85)
+		(start 406.39 102.235)
+		(end 406.39 104.83)
 		(width 0.7)
 		(layer "B.Cu")
@@
 	)
 	(segment
-		(start 410.08 99.89)
-		(end 406.39 103.58)
+		(start 403.7748 105.85)
+		(end 405.37 105.85)
 		(width 0.7)
 		(layer "B.Cu")
@@
 	)
 	(segment
-		(start 270.95 91.94)
-		(end 270.95 93.35)
-		(width 0.7)
-		(layer "B.Cu")
-		(net 107)
-	)
-	(segment
 		(start 214.29 188.35)
 		(end 213.275 188.35)
@@
 	)
 	(segment
-		(start 410.08 91.28)
-		(end 410.08 99.89)
-		(width 0.7)
-		(layer "B.Cu")
-		(net 107)
-	)
-	(segment
 		(start 106.82 207.5)
 		(end 110.11 210.79)
@@
 	)
 	(segment
-		(start 197.4 210.79)
-		(end 220.36 210.79)
+		(start 308.425 89.05)
+		(end 310.95 91.575)
 		(width 0.7)
 		(layer "B.Cu")
@@
 	)
 	(segment
-		(start 403.7748 150.05)
-		(end 403.7 150.05)
+		(start 197.4 210.79)
+		(end 220.36 210.79)
 		(width 0.7)
 		(layer "B.Cu")
@@
 	)
 	(segment
-		(start 407.85 89.05)
-		(end 410.08 91.28)
+		(start 403.7748 150.05)
+		(end 403.7 150.05)
 		(width 0.7)
 		(layer "B.Cu")
@@
 	)
 	(segment
-		(start 336.95 191)
-		(end 312.16 191)
+		(start 336.95 191.425)
+		(end 312.35 191.425)
 		(width 0.2)
 		(layer "F.Cu")
@@
 	)
 	(via
-		(at 336.95 191)
+		(at 336.95 191.425)
 		(size 0.6)
 		(drill 0.3)
@@
 	)
 	(via
-		(at 312.16 191)
+		(at 312.35 191.425)
 		(size 0.6)
 		(drill 0.3)
@@
 	)
 	(segment
-		(start 356.15 191.65)
-		(end 354.69 193.11)
+		(start 304.375 187.6)
+		(end 303.625 188.35)
 		(width 0.2)
 		(layer "B.Cu")
@@
 	)
 	(segment
-		(start 304.375 187.6)
-		(end 303.625 188.35)
+		(start 312.35 191.425)
+		(end 311.2 190.275)
 		(width 0.2)
 		(layer "B.Cu")
@@
 	)
 	(segment
-		(start 311.2 190.04)
-		(end 311.2 188.55)
+		(start 311.2 188.55)
+		(end 310.25 187.6)
 		(width 0.2)
 		(layer "B.Cu")
@@
 	)
 	(segment
-		(start 339.06 193.11)
-		(end 336.95 191)
+		(start 338.635 193.11)
+		(end 336.95 191.425)
 		(width 0.2)
 		(layer "B.Cu")
@@
 	)
 	(segment
-		(start 312.16 191)
-		(end 311.2 190.04)
+		(start 354.69 193.11)
+		(end 338.635 193.11)
 		(width 0.2)
 		(layer "B.Cu")
@@
 	)
 	(segment
-		(start 354.69 193.11)
-		(end 339.06 193.11)
+		(start 356.15 191.65)
+		(end 354.69 193.11)
 		(width 0.2)
 		(layer "B.Cu")
@@
 	)
 	(segment
-		(start 311.2 188.55)
-		(end 310.25 187.6)
+		(start 311.2 190.275)
+		(end 311.2 188.55)
 		(width 0.2)
 		(layer "B.Cu")

Commit message: fix ground plane, update serigraphie
Parts:
- moved R3 3.05 mm to (364.5, 109.4)
- moved R4 3.05 mm to (364.5, 112.4)
- moved R5 3.05 mm to (377.2, 109.4)
- moved R6 3.05 mm to (377.2, 112.4)
- moved C1 2.54 mm to (359.5, 109.4)
- moved C2 2.54 mm to (362.0, 109.4)
- renumbered C2 to C1, C1 to C2, POWER to D70, CAPSLOCK to D71, U1 to Pico, R5 to R1, R6 to R2, R2 to R3, R1 to R4, R4 to R5, R3 to R6
Connections:
- C1 pad 1: Rot CLK -> Rot DT
- C2 pad 1: Rot DT -> Rot CLK
- R3 pad 1: Rot CLK -> Rot DT
- R4 pad 1: Rot DT -> Rot CLK
Routing:
- net Net-(R4-Pad2): track 22.9 -> 26.9 mm
- net Net-(R3-Pad2): track 21.3 -> 20.6 mm
