File: pcb/Anesidora/Anesidora.kicad_sch (KiCad schematic)
At the start: 194 parts, among them J1 Conn_01x06_Socket, SW1 SW_Push_45deg, SW10 SW_Push_45deg, SW11 SW_Push_45deg, SW12 SW_Push_45deg, SW13 SW_Push_45deg, SW14 SW_Push_45deg, SW15 SW_Push_45deg, SW16 SW_Push_45deg, SW17 SW_Push_45deg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

Commit message: add mounting holes
Parts:
- added H11, H12, H13, H14, H15, H16, H17: MountingHole, MountingHole:MountingHole_2.2mm_M2_Pad, symbol Mechanical:MountingHole
